File: power.kicad_sch (KiCad schematic)
At the start: 0 parts

Commit message: rp2350 power + servo rails
Parts:
- added C19, C26, C27, C28: 100nF, PCM_JLCPCB:C_0402, symbol JLCPCB-Capacitors:0402,100nF
- added C20, C21, C22, C23, C30: 10uF, PCM_JLCPCB:C_CASE-A-3216-18(mm), symbol JLCPCB-Capacitors:CASE-A-3216-18(mm),10uF
- added C24, C25: 470uF, PCM_JLCPCB:C_Plugin,D10xL16mm, symbol JLCPCB-Capacitors:Plugin,D10xL16mm,470uF
- added C29: 2.2uF, PCM_JLCPCB:C_0603, symbol JLCPCB-Capacitors:0603,2.2uF
- added D1: Red, PCM_JLCPCB:D_0805, symbol JLCPCB-Diodes:LED,0805,Red
- added D2: Red, PCM_JLCPCB:D_0603, symbol JLCPCB-Diodes:LED,0603,Red
- added J1: USB_C_Receptacle_USB2.0_16P, Connector_USB:USB_C_Receptacle_HCTL_HC-TYPE-C-16P-01A, symbol Connector:USB_C_Receptacle_USB2.0_16P
- added J2: Conn_01x03, Connector_PinHeader_2.54mm:PinHeader_1x03_P2.54mm_Vertical, symbol Connector_Generic:Conn_01x03
- added J3, J4, J5: Conn_01x05, Connector_PinHeader_2.54mm:PinHeader_1x05_P2.54mm_Vertical, symbol Connector_Generic:Conn_01x05
- added R10, R19, R22: 220Ω, PCM_JLCPCB:R_0402, symbol JLCPCB-Resistors:0402,220Ω
- added R11, R8: 5.1kΩ, PCM_JLCPCB:R_0402, symbol JLCPCB-Resistors:0402,5.1kΩ
- added R12, R13, R16, R20, R9: 10kΩ, PCM_JLCPCB:R_0402, symbol JLCPCB-Resistors:0402,10kΩ
- added R14: 33kΩ, PCM_JLCPCB:R_0402, symbol JLCPCB-Resistors:0402,33kΩ
- added R15: 82kΩ, PCM_JLCPCB:R_0603, symbol JLCPCB-Resistors:0603,82kΩ
- added R17, R21: 27kΩ, PCM_JLCPCB:R_0402, symbol JLCPCB-Resistors:0402,10kΩ
- added R18: 680Ω, PCM_JLCPCB:R_0402, symbol JLCPCB-Resistors:0402,680Ω
- added U3: AMS1117-3.3, Package_TO_SOT_SMD:SOT-223-3_TabPin2, symbol Regulator_Linear:AMS1117-3.3
- added U4: TPS2116DRL, Package_TO_SOT_SMD:SOT-583-8, symbol Power_Management:TPS2116DRL
- added U5: SRV05-4, Package_TO_SOT_SMD:SOT-23-6, symbol Power_Protection:SRV05-4
- added U6: ACS712xLCTR-05B, Package_SO:SOIC-8_3.9x4.9mm_P1.27mm, symbol Sensor_Current:ACS712xLCTR-05B
- added U7: LMV321IDBVR, PCM_JLCPCB:SOT-23-5_L3.0-W1.7-P0.95-LS2.8-BR, symbol JLCPCB-Analog:Op-Amp, LMV321IDBVR
- added U8: CJ431, PCM_JLCPCB:SOT-23-3_L2.9-W1.6-P1.90-LS2.8-BR, symbol JLCPCB-Power:Ref, 2-36V, 100mA, CJ431
Connections:
- new net: R16.2, R17.1, U7.1 (+)
- new net: R12.1, R9.2, U4.4 (PR1)
- new net: D1.2, R10.1
- new net: J1.A5 (CC1), R8.1
- new net: R20.2, R21.2, U7.3 (-)
- new net: R19.1, R21.1, U7.4 (OUT)
- new net: D2.2, R22.1
- new net: C27.1, U6.6 (FILTER)
- new net: J1.B5 (CC2), R11.1
- new net +3V3: C21.1, C22.1, R13.1, U3.2 (VO)
- new net +5V: C19.1, C20.1, R18.1, U3.3 (VI), U4.2 (VOUT), U4.7 (VOUT), U6.8 (VCC), U7.5 (V+)
- new net CH1: J2.1 (Pin_1)
- new net CH2: J3.1 (Pin_1)
- new net CH3: J3.2 (Pin_2)
- new net CH4: J3.3 (Pin_3)
- new net CH5: J3.4 (Pin_4)
- new net CH6: J3.5 (Pin_5)
- new net GND: C19.2, C20.2, C21.2, C22.2, C23.2, C24.2, C25.2, C26.2, C27.2, C28.2, C29.2, C30.2, D1.1, D2.1, J1.A1 (GND), J1.A12 (GND), J1.B1 (GND), J1.B12 (GND), J1.S1 (SHIELD), J2.3 (Pin_3), J5.1 (Pin_1), J5.2 (Pin_2), J5.3 (Pin_3), J5.4 (Pin_4), J5.5 (Pin_5), R11.2, R12.2, R15.2, R17.2, R8.2, U3.1 (GND), U4.1 (GND), U5.2 (VN), U6.5 (GND), U7.2 (GND), U8.3 (A)
- new net I_COND: R19.2
- new net I_COND_2_5: R18.2, R20.1, U8.1 (K), U8.2 (R)
- new net I_SRVO_RAW: R16.1, U6.7 (VIOUT)
- new net OTG_FS_VBUS: R14.2, R15.1
- new net PWR_STATUS: R13.2, U4.8 (ST)
- new net USB_D+: J1.A6 (D+), J1.B6 (D+), U5.6 (IO4)
- new net USB_D-: J1.A7 (D-), J1.B7 (D-), U5.1 (IO1)
- new net USB_VBUS: J1.A4 (VBUS), J1.A9 (VBUS), J1.B4 (VBUS), J1.B9 (VBUS), R10.2, R14.1, R9.1, U4.3 (VIN1), U4.5 (MODE), U5.5 (VP)
- new net VBUCK: C28.1, C29.1, C30.1, J4.1 (Pin_1), J4.2 (Pin_2), J4.3 (Pin_3), J4.4 (Pin_4), J4.5 (Pin_5), R22.2, U4.6 (VIN2), U6.3 (IP-), U6.4 (IP-)
- new net VBUCK_IN: C23.1, C24.1, C25.1, C26.1, J2.2 (Pin_2), U6.1 (IP+), U6.2 (IP+)
- no-connect marks 0 -> 4
Other:
- note added: "Servo Bus (CH2-5)"
- note added: "Throttle (CH1) And BEC Power From ESC"
