File: rp-fc2.kicad_sch (KiCad schematic)
At the start: 60 parts, among them CN1 20021521-00010T1LF, SW1 SW_Push, SW2 SW_Push, SW3 SW_Push, U1 W25Q128JVS, U2 W25Q128JVS, U9 RP2350B-QFN80, Y1 Crystal_GND24

Commit message: nrf52833-discrete
Connections:
- net I_COND: now also U9.57 (GPIO46_ADC6)
- net I_COND_2_5: now also U9.58 (GPIO47_ADC7)
- net RP2350_RUN: now reaches C18.1, SW1.2, U9.35 (RUN)
- net RP2350_RUN: now also CN1.10
- net NRF_AUX1: now reaches U9.37 (GPIO29)
- net NRF_AUX2: now reaches U9.38 (GPIO30)
- net NRF_AUX3: now reaches U9.39 (GPIO31)
- net SPI0_MISO: now reaches U9.40 (GPIO32)
- net SPI0_CS: now reaches U9.42 (GPIO33)
- net SPIO_SCK: now reaches U9.43 (GPIO34)
- net SPIO_MOSI: now reaches U9.44 (GPIO35)
- no-connect marks 5 -> 4
Other:
- added sheet IO (io.kicad_sch)
- moved on the sheet: CN1

Commit message: nrf54L BLE module
Parts:
- CN1: footprint easyeda2kicad:IDC-SMD_10P-P1.27_X1270WVS-2X05B-6TV01 -> DigiKey:CONN_3220-10-0100-00_CNC
Changed lines of the file:
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@@
 			)
 		)
-		(property "Footprint" "easyeda2kicad:IDC-SMD_10P-P1.27_X1270WVS-2X05B-6TV01"
+		(property "Footprint" "DigiKey:CONN_3220-10-0100-00_CNC"
 			(at 231.14 111.76 0)
 			(effects
